File: hardware/fk-core-mini-ultra-pro/MINI-ULTRA-PRO.kicad_pcb (KiCad board)
At the start: 2 copper layers, 26.2 x 105.4 mm, 71 parts, among them J1 S2B-PH-SM4-TB, J2 MICRO-USB, J3 RF-SMA-EDGE, J4 CONN-HDR-1x19, J5 CONN-HDR-1x19, J6 CONN-HDR-2x5, J7 RF-SMA-EDGE, M1 MOUNT_HOLE, M2 MOUNT_HOLE, M3 MOUNT_HOLE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

Commit message: Adding logos.
Parts:
- removed M5, M6: FIDUCIAL, RocketScreamKicadLibrary:FIDUCIAL-1MM
- added G***: LOGO, logos:conservify_normal_3500, F.Cu at (134.1, 135.0)
- added G***: LOGO, logos:ngfk_normal_3500, F.Cu at (129.7, 139.8)
- added G***: LOGO, logos:osh_normal_3000, F.Cu at (137.8, 135.0)
Routing:
- net VBAT: track 55.7 -> 54.9 mm
- net (no net): vias 0 -> 5
Other:
- board text added: "v0.1"
