File: hardware/fk-core/fk-core.sch (KiCad schematic (older format))
At the start: 0 parts

Commit message: MUP based board is the primary board now.
Parts:
- added C1, C2: 18pF, RocketScreamKicadLibrary:CAP-0402, symbol CAPACITOR-CERAMIC
- added C10, C11, C14, C16, C17: 4.7uF 10V X5R, RocketScreamKicadLibrary:CAP-0402, symbol CAPACITOR-CERAMIC
- added C12, C13, C3, C4, C6, C7, C8: 100nF, RocketScreamKicadLibrary:CAP-0402, symbol CAPACITOR-CERAMIC
- added C15, C19, C20, C5: 1uF 10V X5R, RocketScreamKicadLibrary:CAP-0402, symbol CAPACITOR-CERAMIC
- added C18: 4.7nF 25V X7R, RocketScreamKicadLibrary:CAP-0402, symbol CAPACITOR-CERAMIC
- added C9: 1uF 50V X5R, RocketScreamKicadLibrary:CAP-0603, symbol CAPACITOR-CERAMIC
- added D1: Orange, RocketScreamKicadLibrary:LED-0603, symbol LED-SINGLE
- added D2: LED-DUAL, RocketScreamKicadLibrary:LED-1615, symbol LED-DUAL
- added D3: PRTR5V0U2X, RocketScreamKicadLibrary:SOT-143B, symbol PRTR5V0U2X
- added D4: PMEG3020CPA, RocketScreamKicadLibrary:SOT-1016, symbol DIODE_DUAL_Schottky
- added D5: Red, RocketScreamKicadLibrary:LED-0603, symbol LED-SINGLE
- added F1: MF-PSMF050X-2, RocketScreamKicadLibrary:MF-PSMF020X, symbol FUSE
- added J1: S2B-PH-SM4-TB, RocketScreamKicadLibrary:S2B-PH-SM4-TB, symbol S2B-PH-SM4-TB
- added J2: MICRO-USB, RocketScreamKicadLibrary:MICRO-USB, symbol MICRO-USB
- added J3, J7: RF-SMA-EDGE, RocketScreamKicadLibrary:RF-SMA-EDGE, symbol RF-SMA-EDGE
- added J4, J5: CONN-HDR-1x19, RocketScreamKicadLibrary:HDR_1x19_Pitch2.54mm_WithoutSilk, symbol CONN-HDR-1x19
- added J6: CONN-HDR-2x5, RocketScreamKicadLibrary:HDR_2x5_Pitch1.27mm, symbol CONN-HDR-2x5
- added L1, L2: BKP1005TS121-T, RocketScreamKicadLibrary:IND-0402, symbol INDUCTOR
- added M1, M2, M3, M4: MOUNT_HOLE, RocketScreamKicadLibrary:HOLE_NPTH_2.2MM, symbol MOUNT_HOLE
- added M5, M6: FIDUCIAL, RocketScreamKicadLibrary:FIDUCIAL-1MM, symbol FIDUCIAL
- added M7: MICROSD, microsd:MICROSD, symbol MICROSD
- added P1: CONN-HDR-MODULE, fk-core-mini-ultra-pro:Socket_Strip_Straight_1x05_Pitch2.54mm, symbol CONN_01X05
- added Q1: 2N7002LT1G, RocketScreamKicadLibrary:SOT-23, symbol MOSFET-N
- added R1, R10, R13: 2K2, RocketScreamKicadLibrary:RES-0402, symbol RESISTOR
- added R11: 100K, RocketScreamKicadLibrary:RES-0402, symbol RESISTOR
- added R12, R4, R8: 10K, RocketScreamKicadLibrary:RES-0402, symbol RESISTOR
- added R14: 1k, RocketScreamKicadLibrary:RES-0402, symbol RESISTOR
- added R15: 180, RocketScreamKicadLibrary:RES-0402, symbol RESISTOR
- added R16: 470R, RocketScreamKicadLibrary:RES-0402, symbol RESISTOR
- added R17, R18: 4.7K, RocketScreamKicadLibrary:RES-0603, symbol RESISTOR
- added R2, R3: 330R, RocketScreamKicadLibrary:RES-0402, symbol RESISTOR
- added R5: 1M, RocketScreamKicadLibrary:RES-0402, symbol RESISTOR
- added R6: 1K18, RocketScreamKicadLibrary:RES-0402, symbol RESISTOR
- added R7: 46K4, RocketScreamKicadLibrary:RES-0402, symbol RESISTOR
- added R9: 2K94, RocketScreamKicadLibrary:RES-0402, symbol RESISTOR
- added SW1: SPNO, RocketScreamKicadLibrary:TS-018, symbol TACT-SWITCH_2Pins
- added U1: ATSAMD21G18A-AU, RocketScreamKicadLibrary:TQFP-48_7x7mm_Pitch0.5mm, symbol ATSAMD21G18A-AU
- added U2: BQ24074RGTT, RocketScreamKicadLibrary:QFN-16_3x3mm, symbol BQ24074
- added U3: RFM95W, RocketScreamKicadLibrary:RFM9xW, symbol RFM9xW
- added U4: MCP1700T-3302E/MB, RocketScreamKicadLibrary:SOT-89, symbol MCP1700T-XXX2E
- added U5: S25FL116K0XMFI041, RocketScreamKicadLibrary:SOIC-8-N, symbol S25FL1xxK0XM
- added U6: MAX1704XX, Housings_DFN_QFN:DFN-8-1EP_2x2mm_Pitch0.5mm, symbol MAX1704XX
- added U7: FGPMMOPA6H, FGPMMOPA6H:FGPMMOPA6H, symbol FGPMMOPA6H
- added Y1: FC-135, RocketScreamKicadLibrary:ABS07, symbol CRYSTAL
Connections:
- net labels added: 3V3, 5V0, A0, A1, A2, A3, A4, A5, AREF, ATN, CHG, D0, D1, D10, D11, D12, D13, D2, D3, D30, D31, D4, D5, D6, D7, D8, D9, GND, MISO, MOSI, PG, RESET, RST, RX_LED, SCK, SCL, SDA, SD_CS, SWCLK, SWDIO, TX_LED, USB+, USB-, USB_ID, VBAT, VBUS, VEXT, VIN, VUSB
- wire segments 0 -> 335
- no-connect marks 0 -> 25
Other:
- note added: "1. All capacitors are NP0/COG 50V unless specified.\n2. All resistors are 62.5mW 1% unless specified."
- note added: "1.27 mm (0.05")"
- note added: "100mA"
- note added: "12.5pF"
- note added: "16Mbit = 2Mbytes"
- note added: "2.54 mm (0.1") breakout"
- note added: "32.768kHz"
- note added: "500mA"
- note added: "BREAKOUT"
- note added: "EN2 EN1"
- note added: "FIDUCIALS"
- note added: "HI HI"
- note added: "HI LOW"
- note added: "I-INPUT LIMIT"
- note added: "LED"
- note added: "LOW HI"
- note added: "LOW LOW"
- note added: "M2.5 size"
- note added: "MCU"
- note added: "MOUNTING"
- note added: "NOTES"
- note added: "POWER MANAGEMENT"
- note added: "RFM95W\n"
- note added: "RX0"
- note added: "RX1"
- note added: "SERIAL FLASH"
- note added: "SWD/JTAG"
- note added: "Set by R6:1.3A"
- note added: "Standby"
- note added: "TX0"
- note added: "TX1"
- note added: "USB-DEVICE"
- note added: "VIN:5-10.5V\n(OVP up to 28V)"

Commit message: Incorporating suggestions from Dave.
* SW1 is awfully close to the RF connection on U7. Can this slide south? Pins 15/15/17/18 are all no connect, having a switch close to that would be easier.
* If you move J7 to the other side of the board, then we won't need a via in the middle of the RF transmission line there.
* R16 is sized to bias A1 at about 3 mA. the default is to toggle on/off when it's locking, then go low when the system is locked. Bumping R16 to ~ 1Kohm will half the current, which might be enough for a high brightness LED.
Done! Thanks!

* Could J3 get flipped so that the RF path stays on the bottom, instead of running through a Via?
Done! I had to narrow and get creative with the A1 trace to route around this, hopefully that's ok.

* Vbackup on U7 might be worthwhile to hookup. the current consumption is pretty low (7 uA) and will let the GPS lock faster when power is applied.
I'll look into doing this. I'm just worried about getting VBAT over to that end of the board, haha.

* If you rotate C1/C2 180 degrees, you can ground both of them at the same via/Ground node.
Good call, where would you put the new via? There's a tight fit right there with the 3v3 to the radio and the edge of the bottom GND fill.

* J1 is an SMT part. Is there one available with through hole mounting pins so the connector doesn't rip off the board?
Good idea, I'll dig around and see if we can find one.

* The BQ24074 supports temp sensing on the battery pack, but the JST connector only has Batt+ and GND. Did you set the charging current on the low side?
* The RFM95 sits right underneath the 32kHz Clock crystal for the SAMD21. The 32kHz is a fairly strong oscillator (32kHz Square wave that goes 0 to 3.3V) and I'm worried that it will couple directly into the RF output of the RFM95 through the Power supply or directly radiated through the board. A 4 layer board with full ground planes would help significantly.

We based our board on an already designed and produced one and these a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
Parts:
- R16: value 470R -> 1k
Connections:
- no-connect marks 25 -> 24
Changed lines of the file:
@@
 LIBS:max1704xx
 LIBS:conn_01x05
-LIBS:ws2812
+LIBS:fk-core-cache
 EELAYER 25 0
 EELAYER END
@@
 	1    0    0    -1
 $EndComp
-NoConn ~ 7450 12350
 NoConn ~ 9300 12650
 Wire Wire Line
@@
 P 6450 12450
 F 0 "R16" H 6450 12550 60  0000 C CNN
-F 1 "470R" H 6450 12350 60  0000 C CNN
+F 1 "1k" H 6450 12350 60  0000 C CNN
 F 2 "RocketScreamKicadLibrary:RES-0402" H 6450 12250 60  0001 C CNN
 F 3 "" H 6450 12450 60  0000 C CNN
@@
 Text Label 3450 10500 0    50   ~ 0
 SD_CS
+$Comp
+L VBAT #PWR?
+U 1 1 58BE06A3
+P 7450 12350
+F 0 "#PWR?" H 7450 12200 50  0001 C CNN
+F 1 "VBAT" H 7450 12490 50  0000 C CNN
+F 2 "" H 7450 12350 60  0000 C CNN
+F 3 "" H 7450 12350 60  0000 C CNN
+	1    7450 12350
+	0    -1   -1   0
+$EndComp
 $EndSCHEMATC
