File: hardware/panelized/fk-core-v0.15-01x04.kicad_pcb (KiCad board)
At the start: 4 copper layers, 121 x 177 mm, 651 parts, among them J1 CONN_01x02, J10 B2B-PH-SM4-TB, J11 RF_UFL_SMD-conservify, J12 CONN_01x02, J13 CONN_01x06, J14 CONN_01x02, J15 RF_UFL_SMD-conservify, J16 Vertical USB, J17 Conn_01x09, J18 Conn_01x01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

Commit message: DFN footprint changes in Core and Panelized Core.
Parts:
- U15 (x4): footprint Package_DFN_QFN:DFN-8-1EP_3x3mm_P0.5mm_EP1.66x2.38mm -> conservify:DFN-8-1EP_3x3mm_P0.5mm_EP1.66x2.38mm
